File: Draytronics Jade.kicad_pcb (KiCad board)
At the start: 2 copper layers, 357.4 x 106.7 mm, 174 parts, among them J1-ISP1 AVR-ISP-6, U1 ATmega32A-PU, Y1 Crystal

Commit message: Added middle standoff for stability
Parts:
- added ?: MountingHole_2.2mm_M2, MountingHole:MountingHole_2.2mm_M2, F.Cu at (221.5, 121.9)
- added ?: MountingHole_2.2mm_M2, MountingHole:MountingHole_2.2mm_M2, F.Cu at (221.5, 25.4)
- added G***: LOGO, logos:qmk-logo, F.Cu at (39.0, 115.4)
- added G***: LOGO, logos:oshw-logo, F.Cu at (37.9, 107.4)
Routing:
- net col11: track 422.0 -> 416.7 mm
- net col12: track 428.1 -> 422.8 mm
- net col13: track 472.1 -> 466.8 mm
- net col14: track 454.8 -> 449.4 mm
- net col8: track 293.4 -> 294.3 mm
Other:
- rule pad_to_mask_clearance: 0.05 -> 0
- board text added: "Designed in the UK by Blake Drayson"
- board text added: "JLCJLCJLCJLC"
- board text removed: "Designed and built in the UK by Blake Drayson"
